File: hw/pedal_board/pedal_board.kicad_pcb (KiCad board)
At the start: 2 copper layers, 94 x 94 mm, 10 parts, among them J1 Conn_01x04, J2 Conn_01x02

Commit message: Added dcdc in board
Parts:
- added U1: dcdc_my3608_mini, dcdc_module_mini:dcdc_module_mini, F.Cu at (215.9, 95.2)
- moved J1 33.7 mm to (149.2, 95.2), turned to 90 degrees
- moved J2 9.44 mm to (197.5, 96.5), turned to 270 degrees
Connections:
- J2 pad 2: /Vin -> Net-(J2-Pad2)
Routing:
- net /Vin: track 8.27 -> 24.3 mm
- net /SCK: track 76.0 -> 65.0 mm, vias 0 -> 1
- net Net-(J2-Pad2): track 0.00 -> 9.54 mm
- net /DT: track 66.1 -> 63.5 mm
