File: hw/pedal_board/pedal_board.sch (KiCad schematic (older format))
At the start: 7 parts, among them J1 Conn_01x04, J2 Conn_01x02

Commit message: Add Panelization test
Parts:
- J2: footprint Connector_PinSocket_2.54mm:PinSocket_1x02_P2.54mm_Vertical -> Connector_JST:JST_XH_B2B-XH-A_1x02_P2.50mm_Vertical
Changed lines of the file:
@@
 F 0 "J2" H 8843 5725 50  0000 C CNN
 F 1 "Conn_01x02" H 8843 5816 50  0000 C CNN
-F 2 "Connector_PinSocket_2.54mm:PinSocket_1x02_P2.54mm_Vertical" H 8925 6050 50  0001 C CNN
+F 2 "Connector_JST:JST_XH_B2B-XH-A_1x02_P2.50mm_Vertical" H 8925 6050 50  0001 C CNN
 F 3 "~" H 8925 6050 50  0001 C CNN
 	1    8925 6050

Commit message: Added dcdc in board
Parts:
- added U1: dcdc_my3608_mini, dcdc_module_mini:dcdc_module_mini, symbol dcdc_module:dcdc_my3608_mini
Connections:
- net GND: now also U1.2 (in_B), U1.4 (out_B)
- net Vin: now also U1.3 (out_A); no longer J2.2 (Pin_2)
- new net: J2.2 (Pin_2), U1.1 (in_A)
Other:
- moved on the sheet: J2
Changed lines of the file:
@@
 L Connector_Generic:Conn_01x02 J2
 U 1 1 603EA83D
-P 8925 6050
-F 0 "J2" H 8843 5725 50  0000 C CNN
-F 1 "Conn_01x02" H 8843 5816 50  0000 C CNN
-F 2 "Connector_JST:JST_XH_B2B-XH-A_1x02_P2.50mm_Vertical" H 8925 6050 50  0001 C CNN
-F 3 "~" H 8925 6050 50  0001 C CNN
-	1    8925 6050
+P 8750 6075
+F 0 "J2" H 8668 5750 50  0000 C CNN
+F 1 "Conn_01x02" H 8668 5841 50  0000 C CNN
+F 2 "Connector_JST:JST_XH_B2B-XH-A_1x02_P2.50mm_Vertical" H 8750 6075 50  0001 C CNN
+F 3 "~" H 8750 6075 50  0001 C CNN
+	1    8750 6075
 	-1   0    0    1
 $EndComp
-Wire Wire Line
-	9125 5950 9550 5950
-Wire Wire Line
-	9125 6050 9325 6050
-Wire Wire Line
-	9325 6050 9325 6200
 $Comp
 L power:GND #PWR0103
 U 1 1 603EC52D
-P 9325 6200
-F 0 "#PWR0103" H 9325 5950 50  0001 C CNN
-F 1 "GND" H 9330 6027 50  0000 C CNN
-F 2 "" H 9325 6200 50  0001 C CNN
-F 3 "" H 9325 6200 50  0001 C CNN
-	1    9325 6200
+P 8950 6200
+F 0 "#PWR0103" H 8950 5950 50  0001 C CNN
+F 1 "GND" H 8955 6027 50  0000 C CNN
+F 2 "" H 8950 6200 50  0001 C CNN
+F 3 "" H 8950 6200 50  0001 C CNN
+	1    8950 6200
 	1    0    0    -1
 $EndComp
-Text Label 9550 5950 2    60   ~ 0
-Vin
 Text Label 7700 3425 2    60   ~ 0
 Vin
@@
 Wire Wire Line
 	7475 3425 7475 4050
+Text Label 10775 5975 2    60   ~ 0
+Vin
+$Comp
+L dcdc_module:dcdc_my3608_mini U1
+U 1 1 605E942C
+P 9725 6075
+F 0 "U1" H 9725 6400 50  0000 C CNN
+F 1 "dcdc_my3608_mini" H 9725 6309 50  0000 C CNN
+F 2 "dcdc_module_mini:dcdc_module_mini" H 9625 6125 50  0001 C CNN
+F 3 "" H 9625 6125 50  0001 C CNN
+	1    9725 6075
+	1    0    0    -1
+$EndComp
+Wire Wire Line
+	8950 5975 9325 5975
+$Comp
+L power:GND #PWR0107
+U 1 1 605EAC3F
+P 9325 6175
+F 0 "#PWR0107" H 9325 5925 50  0001 C CNN
+F 1 "GND" H 9330 6002 50  0000 C CNN
+F 2 "" H 9325 6175 50  0001 C CNN
+F 3 "" H 9325 6175 50  0001 C CNN
+	1    9325 6175
+	1    0    0    -1
+$EndComp
+$Comp
+L power:GND #PWR0108
+U 1 1 605EB174
+P 10125 6175
+F 0 "#PWR0108" H 10125 5925 50  0001 C CNN
+F 1 "GND" H 10130 6002 50  0000 C CNN
+F 2 "" H 10125 6175 50  0001 C CNN
+F 3 "" H 10125 6175 50  0001 C CNN
+	1    10125 6175
+	1    0    0    -1
+$EndComp
+Wire Wire Line
+	10125 5975 10775 5975
+Wire Wire Line
+	8950 6075 8950 6200
 $EndSCHEMATC
